File: XpertRIde_v2.sch (KiCad schematic (older format))
At the start: 44 parts

Commit message: main PCB OK
Parts:
- removed U? (x3): ADG728, Package_SO:TSSOP-16_4.4x5mm_P0.65mm, symbol Analog_Switch:ADG728
- added U2, U3, U4: ADG728, Package_SO:TSSOP-16_4.4x5mm_P0.65mm, symbol perso:ADG728
- C1: renamed from C?; footprint Capacitors_SMD:C_0603_HandSoldering -> Capacitors_SMD:C_0402
- C2, C3, C4, C5, C7: renamed from C?; footprint (none) -> Capacitors_SMD:C_0402
- C6: renamed from C?; footprint (none) -> Capacitors_SMD:C_0603
- J1: renamed from J?; footprint (none) -> perso:Samtec_ESHF_20
- J2: renamed from J?; footprint (none) -> perso:CUI_UJ2-MIBH-4-SMT-TR-67
- J3: renamed from J?; footprint (none) -> perso:Tag_Connect_10
- J4, J5, J6: renamed from J?; footprint (none) -> Wire_Pads:SolderWirePad_single_0-8mmDrill
- J7: renamed from J?; footprint (none) -> Connector_FFC-FPC:TE_84952-5_1x05-1MP_P1.0mm_Horizontal
- R1, R13, R2, R3, R4, R5, R7: renamed from R?; footprint Resistors_SMD:R_0603_HandSoldering -> Resistors_SMD:R_0402
- R10, R11, R12, R14, R15, R16, R17, R18, R19, R20, R21, R8, R9: renamed from R?; footprint (none) -> Resistors_SMD:R_0402
- R6: renamed from R?; value 5k1 -> 5k; footprint Resistors_SMD:R_0603_HandSoldering -> Resistors_SMD:R_0402
- SW1: renamed from SW?; footprint (none) -> perso:DPDT_IP67
- TP1, TP2: renamed from TP?; footprint (none) -> Measurement_Points:Measurement_Point_Round-SMD-Pad_Small
- U1: renamed from U?; value MCP6N11 -> MCP6N11-001
- U5: renamed from U?; footprint (none) -> Package_TO_SOT_SMD:SOT-23-8
Connections:
- net GND is gone; now on net GNDD: R2.2
- net sensorX is gone; now on net SensorX: U1.2 (VIM), U5.7 (B)
- net AMP_OUT: now also U3.8 (D)
- net GNDD: now also J1.20 (Pin_20), U2.14 (GND), U2.15 (A1), U2.16 (A0), U3.14 (GND), U3.15 (A1), U4.14 (GND), U4.16 (A0)
- net Sensor1: now also U2.4 (S1)
- net Sensor2: now also U2.5 (S2)
- net Sensor3: now also U2.6 (S3)
- net Sensor4: now also U2.7 (S4)
- net Sensor5: now also U2.9 (S5)
- net Sensor6: now also U2.10 (S6)
- net Sensor7: now also U2.11 (S7)
- net Sensor8: now also U2.12 (S8)
- net SensorX: now also U2.8 (D)
- net TWI_CLK: now also U2.1 (SCL), U3.1 (SCL), U4.1 (SCL)
- net TWI_SDA: now also U2.3 (SDA), U3.3 (SDA), U4.3 (SDA)
- net VDD: now also U2.13 (VDD), U3.13 (VDD), U4.13 (VDD)
- net digiPot: now also U4.8 (D)
- net at R5.1: now also U2.2 (~RESET)
- net at R12.1: now also U3.9 (S5)
- net at R7.1: now also U3.16 (A0), U3.2 (~RESET)
- net at R8.1: now also U3.4 (S1)
- net at R9.1: now also U3.5 (S2)
- net at R10.1: now also U3.6 (S3)
- net at R11.1: now also U3.7 (S4)
- net at J5.1 (Pin_1): now also SW1.2 (B); no longer SW1.1 (A)
- net at J6.1 (Pin_1): now also SW1.5 (B); no longer SW1.4 (A)
- net at J4.1 (Pin_1): now also SW1.6 (C); no longer SW1.5 (B)
- net at R20.1: now also U4.11 (S7)
- net at R19.1: now also U4.10 (S6)
- net at R18.1: now also U4.9 (S5)
- net at R13.1: now also U4.15 (A1), U4.2 (~RESET)
- net at R14.1: now also U4.4 (S1)
- net at R15.1: now also U4.5 (S2)
- net at R16.1: now also U4.6 (S3)
- net at R17.1: now also U4.7 (S4)
- net at R21.1: now also U4.12 (S8)
- net at C6.2, C7.2, J2.1 (VBUS): now also SW1.3 (C); no longer SW1.2 (B)
- net SWDIO: now reaches J3.2 (Pin_2), TP1.1
- net SDWCLK: now reaches J3.4 (Pin_4), TP2.1
- no-connect marks 13 -> 12
Other:
- moved on the sheet: J4, J5, J6, R12, R18, R19, R20, R21, TP1, TP2
