File: shield/XpertRIde_v2.sch (KiCad schematic (older format))
At the start: 43 parts, among them J1 Conn_01x20, J2 USB_B_Micro, J3 Conn_02x05_Counter_Clockwise, J4 Conn_01x01_Female, J5 Conn_01x01_Female, J6 Conn_01x01_Female, J7 Conn_01x05, SW1 SW_DPDT_x2, U1 MCP6N11-001, U2 ADG728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

Commit message: new design
Parts:
- removed J7: Conn_01x05, Connector_FFC-FPC:TE_84952-5_1x05-1MP_P1.0mm_Horizontal, symbol Connector_Generic:Conn_01x05
- added J7: Conn_02x10_Odd_Even, Pin_Headers:Pin_Header_Straight_2x10_Pitch2.54mm, symbol Connector_Generic:Conn_02x10_Odd_Even
Connections:
- net AMP_OUT: now also J7.3 (Pin_3)
- net GNDD: now also J7.20 (Pin_20)
- net TWI_CLK: now also J7.1 (Pin_1)
- net TWI_SDA: now also J7.2 (Pin_2)
- net VDD: now also J7.19 (Pin_19)
- no-connect marks 12 -> 27
Changed lines of the file:
@@
 Text Notes 4400 3900 0    50   ~ 0
 Amplifier gain selection
-Text Label 9600 2950 2    50   ~ 0
-AMP_OUT
-Text Label 9600 3050 2    50   ~ 0
-TWI_CLK
-Text Label 9600 3150 2    50   ~ 0
-TWI_SDA
-$Comp
-L power:VDD #PWR032
-U 1 1 5EA3130E
-P 9600 3250
-F 0 "#PWR032" H 9600 3100 50  0001 C CNN
-F 1 "VDD" V 9617 3423 50  0000 C CNN
-F 2 "" H 9600 3250 50  0001 C CNN
-F 3 "" H 9600 3250 50  0001 C CNN
-	1    9600 3250
-	0    -1   -1   0
-$EndComp
-$Comp
-L power:GNDD #PWR033
-U 1 1 5EA31465
-P 9600 3350
-F 0 "#PWR033" H 9600 3100 50  0001 C CNN
-F 1 "GNDD" V 9600 3150 50  0000 C CNN
-F 2 "" H 9600 3350 50  0001 C CNN
-F 3 "" H 9600 3350 50  0001 C CNN
-	1    9600 3350
-	0    1    1    0
-$EndComp
-$Comp
-L Connector_Generic:Conn_01x05 J7
-U 1 1 5EA31514
-P 9800 3150
-F 0 "J7" H 9880 3192 50  0000 L CNN
-F 1 "Conn_01x05" H 9880 3101 50  0001 L CNN
-F 2 "Connector_FFC-FPC:TE_84952-5_1x05-1MP_P1.0mm_Horizontal" H 9800 3150 50  0001 C CNN
-F 3 "~" H 9800 3150 50  0001 C CNN
-	1    9800 3150
-	1    0    0    -1
-$EndComp
 Wire Notes Line
 	1350 750  1350 3300
@@
 	6800 6300 10050 6300
 Wire Notes Line
-	9150 2600 10050 2600
-Wire Notes Line
-	10050 2600 10050 3550
-Wire Notes Line
-	10050 3550 9150 3550
-Wire Notes Line
-	9150 3550 9150 2600
-Text Notes 9200 2700 0    50   ~ 0
-Thingy connector
-Wire Notes Line
 	6600 3750 4300 3750
 Wire Notes Line
@@
 L power:PWR_FLAG #FLG0101
 U 1 1 5E9F5533
-P 9400 1400
-F 0 "#FLG0101" H 9400 1475 50  0001 C CNN
-F 1 "PWR_FLAG" H 9400 1573 50  0000 C CNN
-F 2 "" H 9400 1400 50  0001 C CNN
-F 3 "~" H 9400 1400 50  0001 C CNN
-	1    9400 1400
+P 9350 1700
+F 0 "#FLG0101" H 9350 1775 50  0001 C CNN
+F 1 "PWR_FLAG" H 9350 1873 50  0000 C CNN
+F 2 "" H 9350 1700 50  0001 C CNN
+F 3 "~" H 9350 1700 50  0001 C CNN
+	1    9350 1700
 	-1   0    0    1
 $EndComp
@@
 L power:VDD #PWR0102
 U 1 1 5E9FEF84
-P 9400 1400
-F 0 "#PWR0102" H 9400 1250 50  0001 C CNN
-F 1 "VDD" H 9417 1573 50  0000 C CNN
-F 2 "" H 9400 1400 50  0001 C CNN
-F 3 "" H 9400 1400 50  0001 C CNN
-	1    9400 1400
+P 9350 1700
+F 0 "#PWR0102" H 9350 1550 50  0001 C CNN
+F 1 "VDD" H 9367 1873 50  0000 C CNN
+F 2 "" H 9350 1700 50  0001 C CNN
+F 3 "" H 9350 1700 50  0001 C CNN
+	1    9350 1700
 	1    0    0    -1
 $EndComp
@@
 	1    0    0    -1
 $EndComp
+Text Label 9500 2550 2    50   ~ 0
+TWI_CLK
+Text Label 10000 2550 0    50   ~ 0
+TWI_SDA
+Text Label 9500 2650 2    50   ~ 0
+AMP_OUT
+$Comp
+L power:VDD #PWR03
+U 1 1 5EA6D5C0
+P 9500 3450
+F 0 "#PWR03" H 9500 3300 50  0001 C CNN
+F 1 "VDD" V 9517 3623 50  0000 C CNN
+F 2 "" H 9500 3450 50  0001 C CNN
+F 3 "" H 9500 3450 50  0001 C CNN
+	1    9500 3450
+	0    -1   -1   0
+$EndComp
+$Comp
+L power:GNDD #PWR032
+U 1 1 5EA6D621
+P 10000 3450
+F 0 "#PWR032" H 10000 3200 50  0001 C CNN
+F 1 "GNDD" V 10000 3250 50  0000 C CNN
+F 2 "" H 10000 3450 50  0001 C CNN
+F 3 "" H 10000 3450 50  0001 C CNN
+	1    10000 3450
+	0    -1   -1   0
+$EndComp
+NoConn ~ 9500 2750
+NoConn ~ 9500 2850
+NoConn ~ 9500 2950
+NoConn ~ 9500 3050
+NoConn ~ 9500 3150
+NoConn ~ 9500 3250
+NoConn ~ 9500 3350
+NoConn ~ 10000 2650
+NoConn ~ 10000 2750
+NoConn ~ 10000 2850
+NoConn ~ 10000 2950
+NoConn ~ 10000 3050
+NoConn ~ 10000 3150
+NoConn ~ 10000 3250
+NoConn ~ 10000 3350
+Wire Notes Line
+	9050 2250 10400 2250
+Wire Notes Line
+	10400 2250 10400 3600
+Wire Notes Line
+	10400 3600 9050 3600
+Wire Notes Line
+	9050 3600 9050 2250
+Text Notes 9100 2350 0    50   ~ 0
+Thingy connector
+$Comp
+L Connector_Generic:Conn_02x10_Odd_Even J7
+U 1 1 5EAC8CF5
+P 9700 2950
+F 0 "J7" H 9750 3475 50  0000 C CNN
+F 1 "Conn_02x10_Odd_Even" H 9750 3476 50  0001 C CNN
+F 2 "Pin_Headers:Pin_Header_Straight_2x10_Pitch2.54mm" H 9700 2950 50  0001 C CNN
+F 3 "~" H 9700 2950 50  0001 C CNN
+	1    9700 2950
+	1    0    0    -1
+$EndComp

Commit message: fixed switch position
Connections:
- net Sensor5: now also U2.12 (S5); no longer U2.9 (S8)
- net Sensor6: now also U2.11 (S6); no longer U2.10 (S7)
- net Sensor7: now also U2.10 (S7); no longer U2.11 (S6)
- net Sensor8: now also U2.9 (S8); no longer U2.12 (S5)
- net at R12.1: now also U3.12 (S5); no longer U3.9 (S8)
- net at R18.1: now also U4.12 (S5); no longer U4.9 (S8)
- net at R19.1: now also U4.11 (S6); no longer U4.10 (S7)
- net at R20.1: now also U4.10 (S7); no longer U4.11 (S6)
- net at R21.1: now also U4.9 (S8); no longer U4.12 (S5)
Other:
- moved on the sheet: R12, R18, R19, R20, R21
Changed lines of the file:
@@
 EESchema Schematic File Version 4
-LIBS:XpertRIde_v2-cache
-EELAYER 26 0
+EELAYER 30 0
 EELAYER END
 $Descr A4 11693 8268
@@
 	0    -1   -1   0
 $EndComp
+Text Label 3300 2900 2    50   ~ 0
+Sensor8
+Text Label 3300 2800 2    50   ~ 0
+Sensor7
+Text Label 3300 2700 2    50   ~ 0
+Sensor6
 Text Label 3300 2600 2    50   ~ 0
-Sensor8
-Text Label 3300 2700 2    50   ~ 0
-Sensor7
-Text Label 3300 2800 2    50   ~ 0
-Sensor6
-Text Label 3300 2900 2    50   ~ 0
 Sensor5
 Text Label 3300 2500 2    50   ~ 0
@@
 L Device:R R12
 U 1 1 5E9A254B
-P 5150 6000
-F 0 "R12" V 5250 6000 50  0000 C CNN
-F 1 "45k" V 5150 6000 50  0000 C CNN
-F 2 "Resistors_SMD:R_0402" V 5080 6000 50  0001 C CNN
-F 3 "~" H 5150 6000 50  0001 C CNN
-	1    5150 6000
+P 5150 5700
+F 0 "R12" V 5150 5250 50  0000 C CNN
+F 1 "45k" V 5150 5700 50  0000 C CNN
+F 2 "Resistors_SMD:R_0402" V 5080 5700 50  0001 C CNN
+F 3 "~" H 5150 5700 50  0001 C CNN
+	1    5150 5700
 	0    1    1    0
 $EndComp
@@
 L Device:R R18
 U 1 1 5E9E19C1
-P 5400 2950
-F 0 "R18" V 5400 2500 50  0000 C CNN
-F 1 "400k" V 5400 2950 50  0000 C CNN
-F 2 "Resistors_SMD:R_0402" V 5330 2950 50  0001 C CNN
-F 3 "~" H 5400 2950 50  0001 C CNN
-	1    5400 2950
+P 5400 2650
+F 0 "R18" V 5400 2200 50  0000 C CNN
+F 1 "400k" V 5400 2650 50  0000 C CNN
+F 2 "Resistors_SMD:R_0402" V 5330 2650 50  0001 C CNN
+F 3 "~" H 5400 2650 50  0001 C CNN
+	1    5400 2650
 	0    1    1    0
 $EndComp
@@
 L Device:R R19
 U 1 1 5E9F257E
+P 5400 2750
+F 0 "R19" V 5400 2300 50  0000 C CNN
+F 1 "500k" V 5400 2750 50  0000 C CNN
+F 2 "Resistors_SMD:R_0402" V 5330 2750 50  0001 C CNN
+F 3 "~" H 5400 2750 50  0001 C CNN
+	1    5400 2750
+	0    1    1    0
+$EndComp
+$Comp
+L Device:R R20
+U 1 1 5E9F25C8
 P 5400 2850
-F 0 "R19" V 5400 2400 50  0000 C CNN
-F 1 "500k" V 5400 2850 50  0000 C CNN
+F 0 "R20" V 5400 2400 50  0000 C CNN
+F 1 "600k" V 5400 2850 50  0000 C CNN
 F 2 "Resistors_SMD:R_0402" V 5330 2850 50  0001 C CNN
 F 3 "~" H 5400 2850 50  0001 C CNN
@@
 $EndComp
 $Comp
-L Device:R R20
-U 1 1 5E9F25C8
-P 5400 2750
-F 0 "R20" V 5400 2300 50  0000 C CNN
-F 1 "600k" V 5400 2750 50  0000 C CNN
-F 2 "Resistors_SMD:R_0402" V 5330 2750 50  0001 C CNN
-F 3 "~" H 5400 2750 50  0001 C CNN
-	1    5400 2750
-	0    1    1    0
-$EndComp
-$Comp
 L Device:R R21
 U 1 1 5E9F2614
-P 5400 2650
-F 0 "R21" V 5400 2200 50  0000 C CNN
-F 1 "700k" V 5400 2650 50  0000 C CNN
-F 2 "Resistors_SMD:R_0402" V 5330 2650 50  0001 C CNN
-F 3 "~" H 5400 2650 50  0001 C CNN
-	1    5400 2650
+P 5400 2950
+F 0 "R21" V 5400 2500 50  0000 C CNN
+F 1 "700k" V 5400 2950 50  0000 C CNN
+F 2 "Resistors_SMD:R_0402" V 5330 2950 50  0001 C CNN
+F 3 "~" H 5400 2950 50  0001 C CNN
+	1    5400 2950
 	0    1    1    0
 $EndComp
@@
 Connection ~ 5150 2550
 Wire Wire Line
-	5150 2550 5150 2650
-Wire Wire Line
-	5250 2650 5150 2650
-Connection ~ 5150 2650
-Wire Wire Line
-	5150 2650 5150 2750
-Wire Wire Line
 	5250 2750 5150 2750
+Wire Wire Line
+	5250 2850 5150 2850
 Connection ~ 5150 2750
 Wire Wire Line
 	5150 2750 5150 2850
 Wire Wire Line
-	5250 2850 5150 2850
+	5250 2950 5150 2950
 Connection ~ 5150 2850
 Wire Wire Line
 	5150 2850 5150 2950
-Wire Wire Line
-	5250 2950 5150 2950
 Connection ~ 5150 2950
 Wire Wire Line
@@
 	6600 3750 6600 6650
 Wire Wire Line
-	5000 6000 4850 6000
-Wire Wire Line
-	4850 5600 4850 6000
-NoConn ~ 5300 5700
+	4850 5600 4850 5700
 Wire Wire Line
 	4700 6000 4850 6000
-Connection ~ 4850 6000
 $Comp
 L power:GNDD #PWR0101
@@
 	1    0    0    -1
 $EndComp
+Wire Wire Line
+	5150 2550 5150 2650
+Wire Wire Line
+	5250 2650 5150 2650
+Connection ~ 5150 2650
+Wire Wire Line
+	5150 2650 5150 2750
+NoConn ~ 5300 6000
+Wire Wire Line
+	5000 5700 4850 5700
+Connection ~ 4850 5700
+Wire Wire Line
+	4850 5700 4850 6000
 $EndSCHEMATC
